File: hardware/Breadboard_uC.sch (KiCad schematic (older format))
At the start: 35 parts, among them J2 StepPower, U1 Teensy3.2, U2 PD-Micro Module, U3 INA219 Module, U4 MC14490

Commit message: Bugfixes, prepare for 4066
Parts:
- removed D1: 1N5819, Diode_THT:D_DO-41_SOD81_P10.16mm_Horizontal, symbol Diode:1N5819
- removed JU1-4: TeensySpare, Connector_PinHeader_2.54mm:PinHeader_1x06_P2.54mm_Vertical, symbol Connector:Conn_01x06_Male
- removed RU1-1, RU1-2: 2K2, Resistor_THT:R_Axial_DIN0204_L3.6mm_D1.6mm_P7.62mm_Horizontal, symbol Device:R
- added J3: 4066, Connector_PinHeader_2.54mm:PinHeader_1x04_P2.54mm_Vertical, symbol Connector:Conn_01x04_Male
- added JU1-5: U1-VBUS, Connector_PinHeader_2.54mm:PinHeader_1x01_P2.54mm_Vertical, symbol Connector:Conn_01x01_Male
- added JU4-4: Teensy_Spare, Connector_PinHeader_2.54mm:PinHeader_1x08_P2.54mm_Vertical, symbol Connector:Conn_01x08_Male
- added RU11-2: 4K7, Resistor_THT:R_Axial_DIN0204_L3.6mm_D1.6mm_P7.62mm_Horizontal, symbol Device:R
- added RU11-3, RU4-1, RU4-2: 10K, Resistor_THT:R_Axial_DIN0204_L3.6mm_D1.6mm_P7.62mm_Horizontal, symbol Device:R
- added RU2-1: 100, Resistor_THT:R_Axial_DIN0204_L3.6mm_D1.6mm_P7.62mm_Horizontal, symbol Device:R
- added U11: 4066, Package_DIP:DIP-14_W7.62mm, symbol 4xxx:4066
- J2, JU3-1, JU3-2: footprint Connector_Wire:SolderWire-0.25sqmm_1x02_P4.2mm_D0.65mm_OD1.7mm -> Connector_Wire:SolderWire-1sqmm_1x02_P5.4mm_D1.4mm_OD2.7mm
- renumbered RU1-4 to RU1-1, RU1-5 to RU1-2, RU1-6 to RU1-3, RU1-7 to RU1-4, RU1-8 to RU1-5, RU1-10 to RU1-6, RU1-11 to RU1-7, RU1-9 to RU1-8, RU1-3 to RU11-1
Connections:
- net labels added: +5P, TVUSB, VPD-5V, VPD-RAW
- wire segments 248 -> 285
- no-connect marks 14 -> 12
Other:
- moved on the sheet: CU4-2, DU1-1, J2, JU1-1, JU1-2, JU1-3, JU2-1, JU2-2, JU3-1, JU3-2, JU4-1, JU4-2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

Commit message: bugfixes & 4066 functionality
Parts:
- removed J3: 4066, Connector_PinHeader_2.54mm:PinHeader_1x04_P2.54mm_Vertical, symbol Connector:Conn_01x04_Male
- removed RU1-4: 100, Resistor_THT:R_Axial_DIN0204_L3.6mm_D1.6mm_P7.62mm_Horizontal, symbol Device:R
- removed RU11-3: 10K, Resistor_THT:R_Axial_DIN0204_L3.6mm_D1.6mm_P7.62mm_Horizontal, symbol Device:R
- removed unit 1 of U11
- removed unit 4 of U11
- removed unit 3 of U11
- added J17: 4066, Connector_PinHeader_2.54mm:PinHeader_1x04_P2.54mm_Vertical, symbol Connector:Conn_01x04_Male
- added Q4, Q5: BS170, Package_TO_SOT_THT:TO-92_Inline, symbol Transistor_FET:BS170
- added R21, R22: 100, Resistor_THT:R_Axial_DIN0204_L3.6mm_D1.6mm_P7.62mm_Horizontal, symbol Device:R
- added R30, R31: 10K, Resistor_THT:R_Axial_DIN0204_L3.6mm_D1.6mm_P7.62mm_Horizontal, symbol Device:R
- added R33, R36: 4K7, Resistor_THT:R_Axial_DIN0204_L3.6mm_D1.6mm_P7.62mm_Horizontal, symbol Device:R
- added unit 3 of U10
- added unit 4 of U10
- added unit 2 of U10
- J10: renamed from JU2-1; value PDSS/RB0 -> RB0
- J11: renamed from JU4-2; value SW OUT -> SW_OUT
- J12: renamed from JU3-1; value PD_Power -> PD_PWR
- J14: renamed from JU4-4; value Teensy_Spare -> T_Spare
- J15: renamed from JU1-5; value U1-VBUS -> T_VBUS
- J16: renamed from J2; value StepPower -> STEPPWR
- J4: renamed from JU1-3; value Serial -> T_Serial
- J5: renamed from JU1-2; value Rotary Encoder -> Rotary_Enc
- J6: renamed from JU4-3; value PS_Spare1 -> SW_Spare
- J7: renamed from JU1-1; value OLED Display -> OLED
- J8: renamed from JU2-2; value PS_Spare1 -> PS_Spare
- J9: renamed from JU4-1; value SW IN -> SW_IN
- R24: renamed from RU11-2; value 4K7 -> 10K
- R25: renamed from RU11-1; value 4K7 -> 10K
- RL5: renamed from RL6; value HFD4-5 -> HFD4
- RL6: renamed from RL5; value HFD4-5 -> HFD4
- RL7: value HFD4-5 -> HFD4
- RL8: renamed from RL9; value HFD4-5 -> HFD4
- RL9: renamed from RL8; value HFD4-5 -> HFD4
- U8: renamed from U2; value PD-Micro Module -> PD-Micro
- U9: renamed from U3; value INA219 Module -> INA219
- renumbered CU4-2 to C6, DU1-1 to D10, JU3-2 to J13, RU4-1 to R19, RU4-2 to R20, RU2-1 to R23, RU1-1 to R26, RU1-2 to R27, RU1-3 to R28, RU1-5 to R29, RU1-8 to R32, RU1-6 to R34, RU1-7 to R35, U11 to U10, U1 to U11, U4 to U7
Connections:
- net +5P: now also J14.7 (Pin_7)
- net +5V: now also J17.4 (Pin_4), R33.1, R36.1
- net D5: now also R25.1, Q5.1 (D), U10.8; no longer U10.3, U11.7 (5_TX1_PWM)
- net D6: now also R24.1, Q4.1 (D), U10.11; no longer U11.8 (6_PWM)
- net RX: now also J8.3 (Pin_3)
- net SCL: now also J14.6 (Pin_6); no longer J14.8 (Pin_8)
- net SDA: now also J14.5 (Pin_5); no longer J14.7 (Pin_7)
- net TNC1: now also U11.6 (4_RX_PWM); no longer U11.12 (10_TX2_CS_PWM)
- net TNC2: now also U11.28 (21_A7_RX1_CS_PWM); no longer U11.14 (12_DIN)
- net TNC3: now also U11.29 (22_A8_Touch_PWM); no longer U11.28 (21_A7_RX1_CS_PWM)
- net TX: now also J8.2 (Pin_2)
- net PDDTR: now reaches U11.5 (3_TX_PWM)
- net PDDTR: now also R22.1
- net PDRTS: now reaches U11.4 (2)
- net PDRTS: now also R21.1
- net at U8.10 (E6): now also J8.8 (Pin_8); no longer J8.6 (Pin_6)
- net at U8.11 (B4): now also R21.2; no longer J8.7 (Pin_7)
- net at U8.12 (B5): now also R22.2; no longer J8.8 (Pin_8)
- net myMISO: now reaches R27.1, U8.18 (B2)
- net myMOSI: now reaches R26.1, U8.19 (B3)
- net mySCK: now reaches R29.1, U8.20 (B1)
- net PDINT: now reaches R28.1, U8.21 (F7)
- net at U8.5 (SDA): now also J8.4 (Pin_4); no longer J8.2 (Pin_2)
- net at U8.6 (SCL): now also J8.5 (Pin_5); no longer J8.3 (Pin_3)
- net at U8.8 (C6): now also J8.6 (Pin_6); no longer J8.4 (Pin_4)
- net at U8.9 (D7): now also J8.7 (Pin_7); no longer J8.5 (Pin_5)
- net at U11.20 (13_LED_SCK): now also U10.1
- net +3V3: now reaches U11.31 (3.3V)
- net +3V3: now also J14.8 (Pin_8), Q4.2 (G), Q5.2 (G), R30.2, R31.2; no longer J14.6 (Pin_6)
- net PDSS_RB0 renamed RB0
- removed net TNC4: J14.5 (Pin_5), U11.29 (22_A8_Touch_PWM)
- new net: U10.13, U11.14 (12_DIN)
- new net: Q5.3 (S), R30.1, U10.2, U11.7 (5_TX1_PWM)
- new net: Q4.3 (S), R31.1, U11.8 (6_PWM)
- new net: R33.2, U10.9
- new net: R36.2, U10.10
- new net: J17.3 (Pin_3), U10.3
- new net: J17.1 (Pin_1), U10.4
- new net: J17.2 (Pin_2), U10.5
- new net PU_EN: U10.12, U10.6, U11.12 (10_TX2_CS_PWM)
Other:
- moved on the sheet: J10, J12, J13, J15, J16, J4, J5, J6, J7, J8, R23, R24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

Commit message: Updated SPI protocol
Parts:
- added C7: 100uF, symbol Device:CP
- added D10: MBR735, Package_TO_SOT_THT:TO-220-2_Vertical, symbol Diode:MBR735
- added J12: TP_DP, Connector_PinHeader_2.54mm:PinHeader_1x08_P2.54mm_Vertical, symbol Connector:Conn_01x08_Male
- added J13: TP_TNSY, Connector_PinHeader_2.54mm:PinHeader_1x08_P2.54mm_Vertical, symbol Connector:Conn_01x08_Male
- renumbered D10 to D11, J12 to J14, J13 to J15, J14 to J16, J15 to J17, J16 to J18, J17 to J19, R28 to R24, R29 to R25, R24 to R28, R25 to R29
Connections:
- net +3V3: now also J16.5 (Pin_5); no longer J16.8 (Pin_8)
- net +5V: now also J16.6 (Pin_6)
- net C_INT: now also J13.8 (Pin_8)
- net D5: now also J13.6 (Pin_6)
- net D6: now also J13.7 (Pin_7)
- net GND: now also J18.1 (Pin_1), C7.2, J12.1 (Pin_1), J13.1 (Pin_1)
- net PDDTR: now also J12.8 (Pin_8)
- net PDRTS: now also J12.7 (Pin_7)
- net PU_EN: now also J13.5 (Pin_5)
- net SCL: now also J13.3 (Pin_3); no longer J16.6 (Pin_6)
- net SDA: now also J13.2 (Pin_2); no longer J16.5 (Pin_5)
- net TVUSB: now also J16.8 (Pin_8)
- net vsense: now also J18.2 (Pin_2), D10.2 (A); no longer J18.1 (Pin_1), RL9.5
- net CNTR_EN: now reaches U10.13, U11.14 (12_DIN)
- net CNTR_EN: now also J13.4 (Pin_4)
- net MISO: now reaches U11.10 (8_TX3_DIN)
- net MISO: now also R26.2, J12.3 (Pin_3); no longer R27.2
- net PD_INT: now reaches R24.2, U11.13 (11_DOUT)
- net PD_INT: now also J12.6 (Pin_6)
- net SCLK: now reaches R25.2, U11.21 (14_A0_SCK)
- net SCLK: now also J12.4 (Pin_4)
- net MOSI: now reaches U11.9 (7_RX3_DOUT)
- net MOSI: now also R27.2, J12.2 (Pin_2); no longer R26.2
- net at RL9.4: now also RL9.5, C7.1, D10.1 (K); no longer J18.2 (Pin_2)
- net PDINT: no longer names the net of R24.1, U8.21 (F7)
- net RB0 renamed SS
- net SS: now also J12.5 (Pin_5)
- net myMISO: no longer names the net of R27.1, U8.18 (B2)
- net myMOSI: no longer names the net of R26.1, U8.19 (B3)
- net mySCK: no longer names the net of R25.1, U8.20 (B1)
Other:
- moved on the sheet: J16, J18, R24, R25, R26, R27, RL9, U10A

Commit message: Added DMA I2C Monitor
Parts:
- added Q4, Q5: BS170, Package_TO_SOT_THT:TO-92_Inline, symbol Transistor_FET:BS170
- added R24, R25, R31, R33: 10K, Resistor_THT:R_Axial_DIN0204_L3.6mm_D1.6mm_P7.62mm_Horizontal, symbol Device:R
- renumbered J9 to J10, J13 to J11, J10 to J12, J11 to J13, J12 to J8, J8 to J9, Q4 to Q6, Q5 to Q7, R24 to R26, R25 to R27, R26 to R28, R27 to R29, R28 to R30, R29 to R32, R30 to R34, R31 to R35, R32 to R36, R33 to R37, R34 to R38, R35 to R39, R36 to R40
Connections:
- net +3V3: now also Q4.2 (G), Q5.2 (G), R31.2, R33.2
- net +5P: now also U11.33 (Vin)
- net +5V: now also R24.2, R25.2; no longer U11.33 (Vin)
- net SCL: now also Q4.1 (D), R24.1; no longer U11.26 (19_A5_SCL0_Touch)
- net SDA: now also Q5.1 (D), R25.1; no longer U11.25 (18_A4_SDA0_Touch)
- new net T_SCL: Q4.3 (S), R33.1, U11.26 (19_A5_SCL0_Touch)
- new net T_SDA: Q5.3 (S), R31.1, U11.25 (18_A4_SDA0_Touch)
Other:
- moved on the sheet: J11, J16, J8

Commit message: Cleanup main & interrupt driven I2C monitor
Parts:
- removed unit 5 of U10
- added C10: 1n, Capacitor_THT:CP_Radial_Tantal_D5.0mm_P2.50mm, symbol Device:C
- added R36: 1K, Resistor_THT:R_Axial_DIN0204_L3.6mm_D1.6mm_P7.62mm_Horizontal, symbol Device:R
- added U2: 74HC00, Package_DIP:DIP-16_W7.62mm_LongPads, symbol 74xx:74HC00
- added U4: 74HC14, Package_DIP:DIP-16_W7.62mm_LongPads, symbol 74xx:74HC14
- C9: renamed from C7; footprint (none) -> Capacitor_THT:CP_Radial_D6.3mm_P2.50mm
- renumbered C6 to C8, J18 to J16, J16 to J17, J17 to J18, R36 to R37, R37 to R38, R38 to R39, R39 to R40, R40 to R41, RL9 to RL8, RL8 to RL9, U10 to U1, U7 to U10, U8 to U11, U9 to U12, U11 to U13
Connections:
- net D5: now also U2.4, U4.1, U4.13
- net D6: now also U2.12
- net GND: now also C10.2
- net TNC2: now also U13.29 (22_A8_Touch_PWM); no longer U13.28 (21_A7_RX1_CS_PWM)
- net TNC3 renamed SDA_INT
- net SDA_INT: now also U13.28 (21_A7_RX1_CS_PWM), U2.11; no longer U13.29 (22_A8_Touch_PWM)
- new net: U2.1, U4.12
- new net: U2.2, U4.11, U4.8
- new net: U2.3, U2.9
- new net: U2.5, U4.10
- new net: U2.10, U2.6
- new net: U2.13, U2.8
- new net: U4.2, U4.3
- new net: R36.2, U4.4
- new net: U4.6, U4.9
- new net: C10.1, R36.1, U4.5
Other:
- moved on the sheet: C9, D10, J14, J15, J16, RL8, RL9, U12
